File: hardware/V5/kinesisBLE V5.sch (EAGLE design)
At the start: 24 parts, among them X1 JST-XH-02-PIN-ROUND-PAD, X2 JST-XH-02-PIN-ROUND-PAD

Commit message: work in progress
Parts:
- removed R4, R5: 10k, SparkFun-Resistors:10KOHM-HORIZ-1/4W-5%
- added JPL, JPR: (no value), pinhead:PINHD-1X10
- U$4, U$5: value TOPLINKS_STAPELBERG -> MOLEX-39-53-215X-DEVMOLEX-39-53-215X-DEV; device con-molex-39-53:TOPLINKS_STAPELBERG -> nspringkeeb:MOLEX-39-53-215X-DEVMOLEX-39-53-215X-DEV
Connections:
- net N$4 renamed ~RST
- removed net AREF: R4.2, R5.1, U$1.3V@2
- removed net N$19: U$5.P$9
- removed net N$21: MCP23S17.GPB7
- removed net N$24: U$5.P$4
- removed net N$44: U$4.P$5
- removed net N$50: U$4.P$11
- removed net N$54: U$6.P$13
- removed net N$55: U$6.P$11
- removed net N$56: U$6.P$12
- removed net N$57: U$6.P$10
- removed net N$58: U$6.P$9
- removed net N$60: U$6.P$7
- removed net N$61: U$6.P$6
- removed net N$67: U$7.P$1
- removed net N$68: U$7.P$2
- removed net N$75: U$7.P$9
- removed net N$76: U$7.P$10
- removed net N$77: U$7.P$11
- removed net N$78: U$7.P$12
- removed net N$79: U$7.P$13
- net 3V@1: now also U$1.3V@2
- net COL-C: now also JPL.2
- net COL-D: now also JPL.8
- net COL-E: now also JPL.1
- net COL-F: now also JPL.3
- net COL-G: now also JPR.3
- net COL-H: now also JPR.4
- net COL-I: now also JPR.5
- net COL-J: now also JPR.6
- net GND: no longer R5.2
- net N$5: no longer R4.1
- net ROW-6: now also JPL.5, JPR.8
- net ROW-7: now also JPL.4, JPR.7

Commit message: minor reroute, ERC fixes
Parts:
- JPL, JPR: value (none) -> 10
Connections:
- removed net N$5: U$1.USB
Changed lines of the file:
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@@
 <part name="C3" library="SparkFun-Capacitors" deviceset="0.1UF" device="-KIT-EZ-50V-20%" value="0.1uF"/>
 <part name="MCP23S17" library="microchip" library_urn="urn:adsk.eagle:library:294" deviceset="MCP23S17" device="SP" package3d_urn="urn:adsk.eagle:package:20799/2"/>
-<part name="JPR" library="pinhead" library_urn="urn:adsk.eagle:library:325" deviceset="PINHD-1X10" device="" package3d_urn="urn:adsk.eagle:package:22406/2"/>
-<part name="JPL" library="pinhead" library_urn="urn:adsk.eagle:library:325" deviceset="PINHD-1X10" device="" package3d_urn="urn:adsk.eagle:package:22406/2"/>
+<part name="JPR" library="pinhead" library_urn="urn:adsk.eagle:library:325" deviceset="PINHD-1X10" device="" package3d_urn="urn:adsk.eagle:package:22406/2" value="10"/>
+<part name="JPL" library="pinhead" library_urn="urn:adsk.eagle:library:325" deviceset="PINHD-1X10" device="" package3d_urn="urn:adsk.eagle:package:22406/2" value="10"/>
 </parts>
 <sheets>
@@
 </segment>
 </net>
-<net name="N$5" class="0">
-<segment>
-<pinref part="U$1" gate="G$1" pin="USB"/>
-<wire x1="127" y1="30.48" x2="139.7" y2="30.48" width="0.1524" layer="91"/>
-<wire x1="144.78" y1="30.48" x2="139.7" y2="30.48" width="0.1524" layer="91"/>
-<label x="142.24" y="33.02" size="1.778" layer="95"/>
-</segment>
-</net>

Commit message: touches
Parts:
- added AMP: (no value), con-lstb:MA03-1
- added LS1: PS1240P02BT, PS1240P02BT:PS1240P02BT
- added R2: 330, SparkFun-Resistors:330OHM-HORIZ-1/10W-5%
- added R4: 1k, SparkFun-Resistors:1KOHM-HORIZ-1/4W-1%
- added U$8: KSC1815YTA, nspringkeeb:KSC1815YTA
Connections:
- new net N$4: AMP.1, U$8.C
- new net N$5: AMP.2, LS1.1, R4.1
- new net N$7: R2.1, U$8.B
- new net SPK: AMP.3, R2.2, U$1.SCL
- net 3V@1: now also LS1.2, R4.2
- net GND: now also U$8.E
